File: STM32F030_FMRadio.kicad_pcb (KiCad board)
At the start: 2 copper layers, 62 x 27 mm, 20 parts, among them J1 Conn_01x04_Female, J2 Screw_Terminal_01x02, J3 Conn_01x04, J4 Conn_01x05, SW1 Rotary_Encoder_Switch, U1 LP5907MFX-3.3, U2 STM32F030F4Px, U3 TEA5767

Commit message: малкие правки разводки
Routing:
- net GND: track 59.8 -> 56.7 mm
- net Net-(R4-Pad1): track 42.0 -> 40.2 mm
Other:
- board size 62 x 27 mm -> 63 x 29 mm

Commit message: добавлена подтяжка на I2C, перетрассировка
Parts:
- added C10: C, Capacitor_SMD:C_0805_2012Metric, B.Cu at (173.0, 58.0)
- added C11: C, Capacitor_SMD:C_0805_2012Metric, B.Cu at (177.6, 58.0)
- added C9: C, Capacitor_SMD:C_0805_2012Metric, B.Cu at (191.1, 58.4)
- added R5: R, Resistor_SMD:R_0805_2012Metric, B.Cu at (191.1, 54.5)
- added R6: R, Resistor_SMD:R_0805_2012Metric, B.Cu at (174.0, 54.8)
- added R7: R, Resistor_SMD:R_0805_2012Metric, B.Cu at (176.7, 54.8)
- added R8: R, Resistor_SMD:R_0805_2012Metric, B.Cu at (149.4, 59.4)
- added R9: R, Resistor_SMD:R_0805_2012Metric, B.Cu at (146.9, 58.3)
- moved R2 26.1 mm to (186.6, 46.2)
- moved R3 14.1 mm to (180.0, 45.2), turned to 0 degrees
- moved R4 11.6 mm to (180.1, 50.5), turned to 0 degrees
- moved C2 3.54 mm to (150.3, 62.6), turned to 0 degrees
- moved J4 1.76 mm to (147.1, 62.0)
Connections:
- U2 pad 1: Net-(U2-Pad1) -> (no net)
- U2 pad 10: Net-(U2-Pad10) -> (no net)
- U2 pad 11: Net-(U2-Pad11) -> (no net)
- U2 pad 12: Net-(R3-Pad1) -> Net-(C10-Pad2)
- U2 pad 13: Net-(R4-Pad1) -> Net-(C11-Pad2)
- U2 pad 14: Net-(U2-Pad14) -> (no net)
- U2 pad 2: Net-(U2-Pad2) -> (no net)
- U2 pad 3: Net-(U2-Pad3) -> (no net)
- U2 pad 6: Net-(R2-Pad1) -> Net-(C9-Pad1)
- U2 pad 7: Net-(U2-Pad7) -> (no net)
- U2 pad 8: Net-(U2-Pad8) -> (no net)
- U2 pad 9: Net-(U2-Pad9) -> (no net)
- U3 pad 4: Net-(U3-Pad4) -> (no net)
- U3 pad 9: Net-(U3-Pad9) -> (no net)
Routing:
- net Net-(C9-Pad1): track 0.00 -> 35.2 mm, vias 0 -> 2
- net /+3V3: track 86.5 -> 120.9 mm, vias 4 -> 6
- net Net-(R4-Pad1): track 40.2 -> 6.18 mm, vias 2 -> 0
- net Net-(C11-Pad2): track 0.00 -> 31.6 mm
- net Net-(R2-Pad1): track 38.2 -> 9.18 mm, vias 2 -> 0
- net Net-(C10-Pad2): track 0.00 -> 24.5 mm
- net Net-(R3-Pad1): track 36.2 -> 13.5 mm, vias 0 -> 2
- net GND: track 56.7 -> 41.4 mm
- net /SCL: track 37.2 -> 44.7 mm
- net /SDA: track 33.8 -> 39.3 mm
- net /SWCLK: track 19.3 -> 20.2 mm
- net /NRST: track 27.2 -> 28.0 mm
- net /SWDIO: track 16.1 -> 16.9 mm
